File: El_Santo/Kicad_Project/El_Santo/El_Santo.kicad_pcb (KiCad board)
At the start: 2 copper layers, 54.9 x 85.9 mm, 18 parts, among them Q1 2N3904, U1 ICM7555

Commit message: ok
Parts:
- moved R7 77.1 mm to (130.8, 45.1), turned to 0 degrees
- moved R6 68.2 mm to (178.4, 45.7), turned to 180 degrees
- moved S1 31.7 mm to (129.5, 94.0), turned to 270 degrees
- moved R4 26.3 mm to (160.0, 123.2), turned to 0 degrees
- moved U1 25.4 mm to (171.4, 106.0), turned to 0 degrees
- moved R5 19.8 mm to (156.8, 116.2), turned to 270 degrees
- moved R3 19.3 mm to (160.0, 120.0), turned to 0 degrees
- moved BAT1 17.9 mm to (149.2, 114.9), turned to 180 degrees
- moved Q1 12.8 mm to (159.4, 112.4), turned to 180 degrees
- moved C1 8.69 mm to (165.1, 113.7)
- moved R2 5.25 mm to (167.6, 108.6), turned to 180 degrees
- moved C2 3.07 mm to (175.3, 119.4)
- moved D2 2.16 mm to (146.1, 65.2), turned to 180 degrees
- moved R1 0.40 mm to (160.0, 105.4), turned to 0 degrees
Routing:
- net VCC: track 0.00 -> 168.3 mm
- net Net-(D1-Pad1): track 0.00 -> 67.2 mm
- net Net-(C1-Pad1): track 0.00 -> 54.1 mm
- net Net-(R1-Pad2): track 0.00 -> 33.6 mm
- net Net-(D2-Pad2): track 0.00 -> 24.5 mm
- net Net-(C2-Pad1): track 0.00 -> 23.5 mm
- net Net-(D1-Pad2): track 0.00 -> 21.6 mm
- net Net-(BAT1-PadPos): track 0.00 -> 16.0 mm
- net GND: track 0.00 -> 13.5 mm
- net Net-(R3-Pad2): track 0.00 -> 12.1 mm
- net Net-(Q1-Pad2): track 0.00 -> 4.34 mm
- added copper zone on B.Cu, net GND
